Commit message: Added LWR to table.

File: saphari_robot_description/urdf/saphari_robot_description.urdf.xacro (robot description, xacro)
@@ -1,4 +1,7 @@
 <?xml version="1.0"?>
 <robot name="saphari_robot">
+  <include filename="$(find iai_kuka_lwr4_description)/urdf/kuka_lwr_arm.urdf.xacro"/>
+  <include filename="$(find iai_kuka_lwr4_description)/urdf/gazebo.urdf.xacro"/>
+  <include filename="$(find iai_kuka_lwr4_description)/defs/materials.xml"/>
   <link name="ground_plane_frame"/>
   <link name="table_link">
@@ -22,3 +25,6 @@
     <child link="lwr_mounting_frame"/>
   </joint>
+  <kuka_lwr_arm parent="lwr_mounting_frame" name="arm">
+    <origin xyz="0 0 0" rpy="0 0 0"/>
+  </kuka_lwr_arm>
 </robot>

Commit message: Added schnunk flachwechseladapter to urdf.

File: saphari_robot_description/urdf/saphari_robot_description.urdf.xacro (robot description, xacro)
@@ -4,4 +4,5 @@
   <include filename="$(find iai_kuka_lwr4_description)/urdf/gazebo.urdf.xacro"/>
   <include filename="$(find iai_kuka_lwr4_description)/defs/materials.xml"/>
+  <include filename="$(find iai_adapters_description)/urdf/fwk_fwa_050.urdf.xacro"/>
   <link name="ground_plane_frame"/>
   <link name="table_link">
@@ -19,12 +20,15 @@
     <child link="table_link"/>
   </joint>
-  <link name="lwr_mounting_frame"/>
-  <joint name="table_lwr_mounting_offset" type="fixed">
+  <link name="arm_base_link"/>
+  <joint name="table_arm_base_link_offset" type="fixed">
     <origin xyz="0.47 1.029 -0.025" rpy="0 0 0"/>
     <parent link="table_link"/>
-    <child link="lwr_mounting_frame"/>
+    <child link="arm_base_link"/>
   </joint>
-  <kuka_lwr_arm parent="lwr_mounting_frame" name="arm">
+  <kuka_lwr_arm parent="arm_base_link" prefix="">
     <origin xyz="0 0 0" rpy="0 0 0"/>
   </kuka_lwr_arm>
+  <fwk_fwa_050_xacro parent="arm_cabling_adaptor_link" prefix="arm">
+    <origin xyz="0 0 0" rpy="0 0 0" />
+  </fwk_fwa_050_xacro>
 </robot>

Commit message: Added wsg50 to saphari-robot-description.

File: saphari_robot_description/urdf/saphari_robot_description.urdf.xacro (robot description, xacro)
@@ -5,4 +5,5 @@
   <include filename="$(find iai_kuka_lwr4_description)/defs/materials.xml"/>
   <include filename="$(find iai_adapters_description)/urdf/fwk_fwa_050.urdf.xacro"/>
+  <include filename="$(find iai_wsg_50_description)/urdf/wsg_50.urdf.xacro"/>
   <link name="ground_plane_frame"/>
   <link name="table_link">
@@ -32,3 +33,6 @@
     <origin xyz="0 0 0" rpy="0 0 0" />
   </fwk_fwa_050_xacro>
+  <wsg_50_xacro name="gripper" parent="arm_fwk_fwa_050_frame_out">
+    <origin xyz="0 0 0" rpy="0 0 0"/>
+  </wsg_50_xacro>
 </robot>

Commit message: Got rid of unnecesary includes in saphari-robot-description.

File: saphari_robot_description/urdf/saphari_robot_description.urdf.xacro (robot description, xacro)
@@ -2,6 +2,4 @@
 <robot name="saphari_robot">
   <include filename="$(find iai_kuka_lwr4_description)/urdf/kuka_lwr_arm.urdf.xacro"/>
-  <include filename="$(find iai_kuka_lwr4_description)/urdf/gazebo.urdf.xacro"/>
-  <include filename="$(find iai_kuka_lwr4_description)/defs/materials.xml"/>
   <include filename="$(find iai_adapters_description)/urdf/fwk_fwa_050.urdf.xacro"/>
   <include filename="$(find iai_wsg_50_description)/urdf/wsg_50.urdf.xacro"/>
@@ -13,5 +11,7 @@
         <mesh filename="package://saphari_robot_description/meshes/table.stl"/>
       </geometry>
-      <material name="Grey"/>
+      <material name="Grey">
+        <color rgba="0.7 0.7 0.7 1.0"/>
+      </material>
     </visual>
   </link>

Commit message: Added adaptor of firefly cam to urdf of saphari robot.

File: saphari_robot_description/urdf/saphari_robot_description.urdf.xacro (robot description, xacro)
@@ -36,3 +36,19 @@
     <origin xyz="0 0 0" rpy="0 0 0"/>
   </wsg_50_xacro>
+  <link name="firefly_adaptor_link">
+    <visual>
+      <origin rpy="0 0 0" xyz="0 0 0"/>
+      <geometry>
+        <mesh filename="package://saphari_robot_description/meshes/firefly_adaptor.stl"/>
+      </geometry>
+      <material name="Yellow">
+        <color rgba="1.0 0.93 0.7 1.0"/>
+      </material>
+    </visual>
+  </link>
+  <joint name="firefly_adaptor_mounting" type="fixed">
+    <origin xyz="0 0 0" rpy="0 0 0"/>
+    <parent link="gripper_base_link"/>
+    <child link="firefly_adaptor_link"/>
+  </joint>
 </robot>

Commit message: Added blackfly cam to saphari robot description.

File: saphari_robot_description/urdf/saphari_robot_description.urdf.xacro (robot description, xacro)
@@ -8,6 +8,5 @@
     <visual>
       <origin rpy="0 0 0" xyz="0 0 0"/>
-      <geometry>
-        <mesh filename="package://saphari_robot_description/meshes/table.stl"/>
+      <geometry> <mesh filename="package://saphari_robot_description/meshes/table.stl"/>
       </geometry>
       <material name="Grey">
@@ -36,9 +35,9 @@
     <origin xyz="0 0 0" rpy="0 0 0"/>
   </wsg_50_xacro>
-  <link name="firefly_adaptor_link">
+  <link name="blackfly_adaptor_link">
     <visual>
       <origin rpy="0 0 0" xyz="0 0 0"/>
       <geometry>
-        <mesh filename="package://saphari_robot_description/meshes/firefly_adaptor.stl"/>
+        <mesh filename="package://saphari_robot_description/meshes/blackfly_adaptor.stl"/>
       </geometry>
       <material name="Yellow">
@@ -47,8 +46,24 @@
     </visual>
   </link>
-  <joint name="firefly_adaptor_mounting" type="fixed">
+  <joint name="blackfly_adaptor_mounting" type="fixed">
     <origin xyz="0 0 0" rpy="0 0 0"/>
     <parent link="gripper_base_link"/>
-    <child link="firefly_adaptor_link"/>
+    <child link="blackfly_adaptor_link"/>
+  </joint>
+  <link name="blackfly_camera">
+    <visual>
+      <origin rpy="0 0 0" xyz="0 0 0"/>
+      <geometry>
+        <mesh filename="package://saphari_robot_description/meshes/blackfly_camera.stl"/>
+      </geometry>
+      <material name="Grey">
+        <color rgba="0.7 0.7 0.7 1.0"/>
+      </material>
+    </visual>
+  </link>
+  <joint name="blackfly_mounting" type="fixed">
+    <origin xyz="0 -0.0545 0.035" rpy="0 0 3.14"/>
+    <parent link="gripper_base_link"/>
+    <child link="blackfly_camera"/>
   </joint>
 </robot>

Commit message: Corrected mounting of LWR in saphari setup.

File: saphari_robot_description/urdf/saphari_robot_description.urdf.xacro (robot description, xacro)
@@ -4,4 +4,5 @@
   <include filename="$(find iai_adapters_description)/urdf/fwk_fwa_050.urdf.xacro"/>
   <include filename="$(find iai_wsg_50_description)/urdf/wsg_50.urdf.xacro"/>
+  <property name="PI" value="3.1415926535897931" />
   <link name="ground_plane_frame"/>
   <link name="table_link">
@@ -27,5 +28,5 @@
   </joint>
   <kuka_lwr_arm parent="arm_base_link" prefix="">
-    <origin xyz="0 0 0" rpy="0 0 0"/>
+    <origin xyz="0 0 0" rpy="0 0 ${PI / 2.0}"/>
   </kuka_lwr_arm>
   <fwk_fwa_050_xacro parent="arm_cabling_adaptor_link" prefix="arm">

Commit message: Corrected mounting of WSG50 of saphari robot.

File: saphari_robot_description/urdf/saphari_robot_description.urdf.xacro (robot description, xacro)
@@ -34,5 +34,5 @@
   </fwk_fwa_050_xacro>
   <wsg_50_xacro name="gripper" parent="arm_fwk_fwa_050_frame_out">
-    <origin xyz="0 0 0" rpy="0 0 0"/>
+    <origin xyz="0 0 0" rpy="0 0 ${-1*PI*135/180}"/>
   </wsg_50_xacro>
   <link name="blackfly_adaptor_link">

Commit message: Corrected for changes in lwr description.

File: saphari_robot_description/urdf/saphari_robot_description.urdf.xacro (robot description, xacro)
@@ -23,12 +23,12 @@
   <link name="arm_base_link"/>
   <joint name="table_arm_base_link_offset" type="fixed">
-    <origin xyz="0.47 1.029 -0.025" rpy="0 0 0"/>
+    <origin xyz="0.47 1.029 -0.025" rpy="0 0 ${PI / 2.0}"/>
     <parent link="table_link"/>
     <child link="arm_base_link"/>
   </joint>
   <kuka_lwr_arm parent="arm_base_link" prefix="">
-    <origin xyz="0 0 0" rpy="0 0 ${PI / 2.0}"/>
+    <origin xyz="0 0 0" rpy="0 0 0"/>
   </kuka_lwr_arm>
-  <fwk_fwa_050_xacro parent="arm_cabling_adaptor_link" prefix="arm">
+  <fwk_fwa_050_xacro parent="arm_flange_link" prefix="arm">
     <origin xyz="0 0 0" rpy="0 0 0" />
   </fwk_fwa_050_xacro>

Commit message: External camera calibration as calculated with halcom.

File: saphari_robot_description/urdf/saphari_robot_description.urdf.xacro (robot description, xacro)
@@ -5,4 +5,5 @@
   <include filename="$(find iai_wsg_50_description)/urdf/wsg_50.urdf.xacro"/>
   <property name="PI" value="3.1415926535897931" />
+  <!-- FURNITURE AND SCENE -->
   <link name="ground_plane_frame"/>
   <link name="table_link">
@@ -21,4 +22,5 @@
     <child link="table_link"/>
   </joint>
+  <!-- LWR AND GRIPPER -->
   <link name="arm_base_link"/>
   <joint name="table_arm_base_link_offset" type="fixed">
@@ -36,4 +38,5 @@
     <origin xyz="0 0 0" rpy="0 0 ${-1*PI*135/180}"/>
   </wsg_50_xacro>
+  <!-- WRIST CAM WITH MOUNTING -->
   <link name="blackfly_adaptor_link">
     <visual>
@@ -68,3 +71,17 @@
     <child link="blackfly_camera"/>
   </joint>
+  <!-- CAMERA CALIBRATION -->
+  <!-- TO BE SIMPLIFIED INTO ONE LINK-JOINT COMBO -->
+  <link name="optical_frame_x" />
+  <joint name="optical_joint_x" type="fixed">
+    <origin xyz="0.000836 -0.053028 0.073603" rpy="0.007552 6.274592 3.141201"/>
+    <parent link="gripper_base_link" />
+    <child link="optical_frame_x" />
+  </joint>
+  <link name="optical_frame" />
+  <joint name="optical_joint" type="fixed">
+    <origin xyz="0.0 0.0 0.0" rpy="0.0 0.0 ${PI}" />
+    <parent link="optical_frame_x" />
+    <child link="optical_frame" />
+  </joint>
 </robot>

Commit message: Added pickup-zone, target-basket, and mounted screen to saphari urdf.

File: saphari_robot_description/urdf/saphari_robot_description.urdf.xacro (robot description, xacro)
@@ -21,4 +21,114 @@
     <parent link="ground_plane_frame"/>
     <child link="table_link"/>
+  </joint>
+  <link name="screenholder_1_link">
+    <visual>
+      <origin xyz="0.04 0.165 0.02" rpy="0 0 0" />
+      <geometry>
+        <box size="0.08 0.325 0.04" />
+      </geometry>
+      <material name="Grey"/>
+    </visual>
+  </link>
+  <joint name="screenholder_mounting_joint" type="fixed">
+    <!-- TODO: verify y-component of this translation! -->
+    <origin xyz="1.19 0.6 -0.08" rpy="0 0 0"/>
+    <parent link="table_link"/>
+    <child link="screenholder_1_link"/>
+  </joint>
+  <link name="screenholder_2_link">
+    <visual>
+      <origin xyz="0.04 0.02 0.1625" rpy="0 0 0" />
+      <geometry>
+        <box size="0.08 0.04 0.325" />
+      </geometry>
+      <material name="Grey"/>
+    </visual>
+  </link>
+  <joint name="screenholder_1_joint" type="fixed">
+    <origin xyz="0.0 ${0.325 - 0.045 - 0.04} 0.04" rpy="0 0 0"/>
+    <parent link="screenholder_1_link"/>
+    <child link="screenholder_2_link"/>
+  </joint>
+  <link name="screenholder_3_link">
+    <visual>
+      <origin xyz="0 -0.01 ${0.05/2}" rpy="0 0 0" />
+      <geometry>
+        <cylinder radius="0.01" length="0.05"/>
+      </geometry>
+      <material name="Black">
+        <color rgba="0 0 0 1.0"/>
+      </material>
+    </visual>
+  </link>
+  <joint name="screenholder_2_joint" type="fixed">
+    <origin xyz="${0.08/2} 0.0 ${0.325 - 0.05 - 0.05/2}" rpy="0 0 0"/>
+    <parent link="screenholder_2_link"/>
+    <child link="screenholder_3_link"/>
+  </joint>
+  <link name="screenholder_4_link">
+    <visual>
+      <origin xyz="0 ${-0.06/2} ${0.04/2}" rpy="0 0 0" />
+      <geometry>
+        <box size="0.01 0.06 0.04" />
+      </geometry>
+      <material name="Black">
+        <color rgba="0 0 0 1.0"/>
+      </material>
+    </visual>
+  </link>
+  <joint name="screenholder_3_joint" type="fixed">
+    <origin xyz="0 ${-0.02/2} 0.005" rpy="0 0 ${-45*PI/180}"/>
+    <parent link="screenholder_3_link"/>
+    <child link="screenholder_4_link"/>
+  </joint>
+  <link name="screen">
+    <visual>
+      <origin xyz="0 ${-0.045/2} ${0.32/2}" rpy="0 0 0" />
+      <geometry>
+        <box size="0.55 0.045 0.32" />
+      </geometry>
+      <material name="Black">
+        <color rgba="0 0 0 1.0"/>
+      </material>
+    </visual>
+  </link>
+  <joint name="screen_mounting_joint" type="fixed">
+    <!-- TODO: verify the z-component of this translation -->
+    <origin xyz="0 -0.06 -0.18" rpy="0 0 0"/>
+    <parent link="screenholder_4_link"/>
+    <child link="screen"/>
+  </joint>
+  <link name="instrument_pad">
+    <visual>
+      <origin xyz="0.28 0.135 0.001" rpy="0 0 0" />
+      <geometry>
+        <box size="0.56 0.27 0.002" />
+      </geometry>
+      <material name="LightBlue">
+        <color rgba="${80/255} ${100/255} ${210/255} 1.0"/>
+      </material>
+    </visual>
+  </link>
+  <joint name="instrument_pad_to_table_offset" type="fixed">
+    <origin xyz="0 0.26 0" rpy="0 0 0"/>
+    <parent link="table_link"/>
+    <child link="instrument_pad"/>
+  </joint>
+  <link name="sorting_basket">
+    <visual>
+      <origin xyz="0.2025 0.125 0.02" rpy="0 0 0" />
+      <geometry>
+        <box size="0.405 0.25 0.04" />
+      </geometry>
+      <material name="Silver">
+        <color rgba="${160/255} ${160/255} ${190/255} 1.0"/>
+      </material>
+    </visual>
+  </link>
+  <joint name="sorting_basket_to_table_offset" type="fixed">
+    <origin xyz="0.72 0.255 0" rpy="0 0 ${PI*39/180}"/>
+    <parent link="table_link"/>
+    <child link="sorting_basket"/>
   </joint>
   <!-- LWR AND GRIPPER -->

Commit message: Merge separate urdf for SAPHARI table.

File: saphari_robot_description/urdf/saphari_robot_description.urdf.xacro (robot description, xacro)
@@ -4,100 +4,11 @@
   <include filename="$(find iai_adapters_description)/urdf/fwk_fwa_050.urdf.xacro"/>
   <include filename="$(find iai_wsg_50_description)/urdf/wsg_50.urdf.xacro"/>
+  <include filename="$(find saphari_robot_description)/urdf/saphari_table.urdf.xacro"/>
   <property name="PI" value="3.1415926535897931" />
   <!-- FURNITURE AND SCENE -->
-  <link name="ground_plane_frame"/>
-  <link name="table_link">
-    <visual>
-      <origin rpy="0 0 0" xyz="0 0 0"/>
-      <geometry> <mesh filename="package://saphari_robot_description/meshes/table.stl"/>
-      </geometry>
-      <material name="Grey">
-        <color rgba="0.7 0.7 0.7 1.0"/>
-      </material>
-    </visual>
-  </link>
-  <joint name="ground_plane_to_table_offset" type="fixed">
+  <link name="map"/>
+  <saphari_table parent="map">
     <origin xyz="0 0 0.89" rpy="0 0 0"/>
-    <parent link="ground_plane_frame"/>
-    <child link="table_link"/>
-  </joint>
-  <link name="screenholder_1_link">
-    <visual>
-      <origin xyz="0.04 0.165 0.02" rpy="0 0 0" />
-      <geometry>
-        <box size="0.08 0.325 0.04" />
-      </geometry>
-      <material name="Grey"/>
-    </visual>
-  </link>
-  <joint name="screenholder_mounting_joint" type="fixed">
-    <!-- TODO: verify y-component of this translation! -->
-    <origin xyz="1.19 0.6 -0.08" rpy="0 0 0"/>
-    <parent link="table_link"/>
-    <child link="screenholder_1_link"/>
-  </joint>
-  <link name="screenholder_2_link">
-    <visual>
-      <origin xyz="0.04 0.02 0.1625" rpy="0 0 0" />
-      <geometry>
-        <box size="0.08 0.04 0.325" />
-      </geometry>
-      <material name="Grey"/>
-    </visual>
-  </link>
-  <joint name="screenholder_1_joint" type="fixed">
-    <origin xyz="0.0 ${0.325 - 0.045 - 0.04} 0.04" rpy="0 0 0"/>
-    <parent link="screenholder_1_link"/>
-    <child link="screenholder_2_link"/>
-  </joint>
-  <link name="screenholder_3_link">
-    <visual>
-      <origin xyz="0 -0.01 ${0.05/2}" rpy="0 0 0" />
-      <geometry>
-        <cylinder radius="0.01" length="0.05"/>
-      </geometry>
-      <material name="Black">
-        <color rgba="0 0 0 1.0"/>
-      </material>
-    </visual>
-  </link>
-  <joint name="screenholder_2_joint" type="fixed">
-    <origin xyz="${0.08/2} 0.0 ${0.325 - 0.05 - 0.05/2}" rpy="0 0 0"/>
-    <parent link="screenholder_2_link"/>
-    <child link="screenholder_3_link"/>
-  </joint>
-  <link name="screenholder_4_link">
-    <visual>
-      <origin xyz="0 ${-0.06/2} ${0.04/2}" rpy="0 0 0" />
-      <geometry>
-        <box size="0.01 0.06 0.04" />
-      </geometry>
-      <material name="Black">
-        <color rgba="0 0 0 1.0"/>
-      </material>
-    </visual>
-  </link>
-  <joint name="screenholder_3_joint" type="fixed">
-    <origin xyz="0 ${-0.02/2} 0.005" rpy="0 0 ${-45*PI/180}"/>
-    <parent link="screenholder_3_link"/>
-    <child link="screenholder_4_link"/>
-  </joint>
-  <link name="screen">
-    <visual>
-      <origin xyz="0 ${-0.045/2} ${0.32/2}" rpy="0 0 0" />
-      <geometry>
-        <box size="0.55 0.045 0.32" />
-      </geometry>
-      <material name="Black">
-        <color rgba="0 0 0 1.0"/>
-      </material>
-    </visual>
-  </link>
-  <joint name="screen_mounting_joint" type="fixed">
-    <!-- TODO: verify the z-component of this translation -->
-    <origin xyz="0 -0.06 -0.18" rpy="0 0 0"/>
-    <parent link="screenholder_4_link"/>
-    <child link="screen"/>
-  </joint>
+  </saphari_table>
   <link name="instrument_pad">
     <visual>
