Commit message: Added kinect calibration as sent around by Rico.

File: saphari_robot_description/urdf/saphari_map.urdf.xacro (robot description, xacro)
@@ -2,5 +2,5 @@
 <robot xmlns:xacro="http://www.ros.org/wiki/xacro" name="saphari_map">
   <include filename="$(find iai_kinect_description)/urdf/kinect.urdf.xacro"/>
-  <macro name="saphari_map" params="map_frame">
+  <macro name="saphari_map" params="map_frame kinect_calib_parent_frame kinect_calib_frame *kinect_calib">
     <link name="${map_frame}"/>
     <link name="wall">
@@ -92,8 +92,13 @@
       <child link="kinect_mounting_5_link"/>
     </joint>
-    <!-- TODO: correct calibration! so far only visually pleasing -->
     <kinect name="kinect" parent="kinect_mounting_5_link">
       <origin xyz="0.03 -0.01 ${-0.03 -0.02 -0.015}" rpy="0 0 ${-90*PI/180}"/>
     </kinect>
+    <link name="${kinect_calib_frame}"/>
+    <joint name="kinect_calibration" type="fixed">
+      <insert_block name="kinect_calib"/>
+      <parent link="${kinect_calib_parent_frame}"/>
+      <child link="${kinect_calib_frame}"/>
+    </joint>
   </macro>
 </robot>

File: saphari_robot_description/urdf/saphari_setup_description.urdf.xacro (robot description, xacro)
@@ -8,14 +8,11 @@
   <property name="PI" value="3.1415926535897931" />
   <!-- FURNITURE AND SCENE -->
-  <saphari_map map_frame="map"/>
+  <saphari_map map_frame="map" kinect_calib_parent_frame="arm_base_link" kinect_calib_frame="openni_depth_frame">
+    <origin xyz="0.286111 -1.14642 1.34476" rpy="-2.1339635300413633 -0.07999807283761096 0.9304591444760072"/>
+    <!-- ORIGINAL QUATERNION: 0.773385 0.409824 -0.185113 -0.446826 -->
+  </saphari_map>
   <saphari_table parent="map">
     <origin xyz="0 0 0.89" rpy="0 0 0"/>
   </saphari_table>
-  <!--link name="measurement_frame"/>
-  <joint name="measurement" type="fixed">
-    <origin xyz="0.6 0.75 0" rpy="0 0 0"/>
-    <parent link="table_link"/>
-    <child link="measurement_frame"/>
-  </joint-->
   <link name="instrument_pad">
     <visual>
@@ -65,5 +62,4 @@
   <wsg_50_xacro name="gripper" parent="arm_fwk_fwa_050_frame_out">
     <origin xyz="0 0 0" rpy="0 0 ${PI*45/180}"/>
-    <!--origin xyz="0 0 0" rpy="0 0 ${-1*PI*135/180}"/-->
   </wsg_50_xacro>
   <!-- WRIST CAM WITH MOUNTING -->
