Commit message: Added wall and wall-mounted kinect to urdf of saphari setup.

File: saphari_robot_description/urdf/saphari_setup_description.urdf.xacro (robot description, xacro)
@@ -5,10 +5,17 @@
   <include filename="$(find iai_wsg_50_description)/urdf/wsg_50.urdf.xacro"/>
   <include filename="$(find saphari_robot_description)/urdf/saphari_table.urdf.xacro"/>
+  <include filename="$(find saphari_robot_description)/urdf/saphari_map.urdf.xacro"/>
   <property name="PI" value="3.1415926535897931" />
   <!-- FURNITURE AND SCENE -->
-  <link name="map"/>
+  <saphari_map map_frame="map"/>
   <saphari_table parent="map">
     <origin xyz="0 0 0.89" rpy="0 0 0"/>
   </saphari_table>
+  <!--link name="measurement_frame"/>
+  <joint name="measurement" type="fixed">
+    <origin xyz="0.6 0.75 0" rpy="0 0 0"/>
+    <parent link="table_link"/>
+    <child link="measurement_frame"/>
+  </joint-->
   <link name="instrument_pad">
     <visual>

Commit message: Mirrored rotation of gripper to improve look-at configuration.

File: saphari_robot_description/urdf/saphari_setup_description.urdf.xacro (robot description, xacro)
@@ -64,5 +64,6 @@
   </fwk_fwa_050_xacro>
   <wsg_50_xacro name="gripper" parent="arm_fwk_fwa_050_frame_out">
-    <origin xyz="0 0 0" rpy="0 0 ${-1*PI*135/180}"/>
+    <origin xyz="0 0 0" rpy="0 0 ${PI*45/180}"/>
+    <!--origin xyz="0 0 0" rpy="0 0 ${-1*PI*135/180}"/-->
   </wsg_50_xacro>
   <!-- WRIST CAM WITH MOUNTING -->

Commit message: Switched to new holder of blackfly and protector of wsg in saphari-robot-description.

File: saphari_robot_description/urdf/saphari_setup_description.urdf.xacro (robot description, xacro)
@@ -68,19 +68,51 @@
   </wsg_50_xacro>
   <!-- WRIST CAM WITH MOUNTING -->
-  <link name="blackfly_adaptor_link">
+  <link name="gripper_top_protector">
     <visual>
       <origin rpy="0 0 0" xyz="0 0 0"/>
       <geometry>
-        <mesh filename="package://saphari_robot_description/meshes/blackfly_adaptor.stl"/>
+        <mesh filename="package://saphari_robot_description/meshes/top_protector.stl" scale="0.001 0.001 0.001"/>
       </geometry>
-      <material name="Yellow">
-        <color rgba="1.0 0.93 0.7 1.0"/>
+      <material name="Blue">
+        <color rgba="0.0 0.0 1.0 1.0"/>
       </material>
     </visual>
   </link>
-  <joint name="blackfly_adaptor_mounting" type="fixed">
-    <origin xyz="0 0 0" rpy="0 0 0"/>
+  <link name="gripper_bottom_protector">
+    <visual>
+      <origin rpy="0 0 0" xyz="0 0 0"/>
+      <geometry>
+        <mesh filename="package://saphari_robot_description/meshes/bottom_protector.stl" scale="0.001 0.001 0.001"/>
+      </geometry>
+      <material name="Blue">
+        <color rgba="0.0 0.0 1.0 1.0"/>
+      </material>
+    </visual>
+  </link>
+  <link name="blackfly_holder">
+    <visual>
+      <origin rpy="0 0 0" xyz="0 0 0"/>
+      <geometry>
+        <mesh filename="package://saphari_robot_description/meshes/camera_mount_blackfly.stl" scale="0.001 0.001 0.001"/>
+      </geometry>
+      <material name="Blue">
+        <color rgba="0.0 0.0 1.0 1.0"/>
+      </material>
+    </visual>
+  </link>
+  <joint name="gripper_top_protector_mounting" type="fixed">
+    <origin xyz="0 0 0" rpy="${-90*PI/180} 0 ${PI}"/>
     <parent link="gripper_base_link"/>
-    <child link="blackfly_adaptor_link"/>
+    <child link="gripper_top_protector"/>
+  </joint>
+  <joint name="gripper_bottom_protector_mounting" type="fixed">
+    <origin xyz="0 0 0.07" rpy="${90*PI/180} 0 0"/>
+    <parent link="gripper_base_link"/>
+    <child link="gripper_bottom_protector"/>
+  </joint>
+  <joint name="blackfly_holder_mounting" type="fixed">
+    <origin xyz="0 0 0" rpy="${-90*PI/180} 0 0"/>
+    <parent link="gripper_base_link"/>
+    <child link="blackfly_holder"/>
   </joint>
   <link name="blackfly_camera">

Commit message: New extrinsic calibration of blackfly, as calculated by halcon.

File: saphari_robot_description/urdf/saphari_setup_description.urdf.xacro (robot description, xacro)
@@ -136,6 +136,7 @@
   <link name="optical_frame_x" />
   <joint name="optical_joint_x" type="fixed">
-    <origin xyz="0.000836 -0.053028 0.073603" rpy="0.007552 6.274592 3.141201"/>
-    <parent link="gripper_base_link" />
+    <origin xyz="0.041576 -0.037009 0.142994"
+            rpy="0.002172 6.277456 4.001921"/>
+    <parent link="arm_7_link" />
     <child link="optical_frame_x" />
   </joint>

Commit message: added meshes for basket and table

File: saphari_robot_description/urdf/saphari_setup_description.urdf.xacro (robot description, xacro)
@@ -33,7 +33,7 @@
   <link name="sorting_basket">
     <visual>
-      <origin xyz="0.2025 0.125 0.02" rpy="0 0 0" />
+      <origin xyz="0.2025 0.0 0.02" rpy="0 0 0" />
       <geometry>
-        <box size="0.405 0.25 0.04" />
+        <mesh filename="package://saphari_robot_description/meshes/saphari_basket.dae"/>
       </geometry>
       <material name="Silver">

File: saphari_robot_description/urdf/saphari_table.urdf.xacro (robot description, xacro)
@@ -6,5 +6,5 @@
       <visual>
         <origin rpy="0 0 0" xyz="0 0 0"/>
-        <geometry> <mesh filename="package://saphari_robot_description/meshes/table.stl"/>
+        <geometry> <mesh filename="package://saphari_robot_description/meshes/table.dae"/>
         </geometry>
         <material name="Grey">

Commit message: Removed instrument pad from urdf.

File: saphari_robot_description/urdf/saphari_setup_description.urdf.xacro (robot description, xacro)
@@ -15,20 +15,4 @@
     <origin xyz="0 0 0.89" rpy="0 0 0"/>
   </saphari_table>
-  <link name="instrument_pad">
-    <visual>
-      <origin xyz="0.28 0.135 0.001" rpy="0 0 0" />
-      <geometry>
-        <box size="0.56 0.27 0.002" />
-      </geometry>
-      <material name="LightBlue">
-        <color rgba="${80/255} ${100/255} ${210/255} 1.0"/>
-      </material>
-    </visual>
-  </link>
-  <joint name="instrument_pad_to_table_offset" type="fixed">
-    <origin xyz="0 0.26 0" rpy="0 0 0"/>
-    <parent link="table_link"/>
-    <child link="instrument_pad"/>
-  </joint>
   <link name="sorting_basket">
     <visual>

Commit message: Correct height of sorting basket in urdf.
Correct height of sorting basket in urdf.

File: saphari_robot_description/urdf/saphari_setup_description.urdf.xacro (robot description, xacro)
@@ -17,5 +17,5 @@
   <link name="sorting_basket">
     <visual>
-      <origin xyz="0.2025 0.0 0.02" rpy="0 0 0" />
+      <origin xyz="0.2025 0.0 0.0" rpy="0 0 0" />
       <geometry>
         <mesh filename="package://saphari_robot_description/meshes/saphari_basket.dae"/>

Commit message: Changed name of blackly optical-frame to wrist_optical_frame.

File: saphari_robot_description/urdf/saphari_setup_description.urdf.xacro (robot description, xacro)
@@ -114,16 +114,16 @@
   <!-- CAMERA CALIBRATION -->
   <!-- TO BE SIMPLIFIED INTO ONE LINK-JOINT COMBO -->
-  <link name="optical_frame_x" />
+  <link name="wrist_optical_frame_x" />
   <joint name="optical_joint_x" type="fixed">
     <origin xyz="0.041576 -0.037009 0.142994"
             rpy="0.002172 6.277456 4.001921"/>
     <parent link="arm_7_link" />
-    <child link="optical_frame_x" />
+    <child link="wrist_optical_frame_x" />
   </joint>
-  <link name="optical_frame" />
+  <link name="wrist_optical_frame" />
   <joint name="optical_joint" type="fixed">
     <origin xyz="0.0 0.0 0.0" rpy="0.0 0.0 ${PI}" />
-    <parent link="optical_frame_x" />
-    <child link="optical_frame" />
+    <parent link="wrist_optical_frame_x" />
+    <child link="wrist_optical_frame" />
   </joint>
 </robot>

Commit message: Corrected visual offset of basket in urdf.

File: saphari_robot_description/urdf/saphari_setup_description.urdf.xacro (robot description, xacro)
@@ -17,5 +17,5 @@
   <link name="sorting_basket">
     <visual>
-      <origin xyz="0.2025 0.0 0.0" rpy="0 0 0" />
+      <origin xyz="0.2025 0.125 0.0" rpy="0 0 0" />
       <geometry>
         <mesh filename="package://saphari_robot_description/meshes/saphari_basket.dae"/>

Commit message: Corrected orientation of the camera pose. Artificially introduced rot of 180deg after calib was a misunderstanding.

File: saphari_robot_description/urdf/saphari_setup_description.urdf.xacro (robot description, xacro)
@@ -114,15 +114,9 @@
   <!-- CAMERA CALIBRATION -->
   <!-- TO BE SIMPLIFIED INTO ONE LINK-JOINT COMBO -->
-  <link name="wrist_optical_frame_x" />
-  <joint name="optical_joint_x" type="fixed">
+  <link name="wrist_optical_frame" />
+  <joint name="optical_joint" type="fixed">
     <origin xyz="0.041576 -0.037009 0.142994"
             rpy="0.002172 6.277456 4.001921"/>
     <parent link="arm_7_link" />
-    <child link="wrist_optical_frame_x" />
-  </joint>
-  <link name="wrist_optical_frame" />
-  <joint name="optical_joint" type="fixed">
-    <origin xyz="0.0 0.0 0.0" rpy="0.0 0.0 ${PI}" />
-    <parent link="wrist_optical_frame_x" />
     <child link="wrist_optical_frame" />
   </joint>
